Commit message: add: fake hardware tags and robot_id parameters in urdf
Add:
 - 'use_fake_hardware' xacro arg
 - 'robot_id' xacro arg
 - 'plugin_name' xacro arg

File: fd_description/config/fd.config.xacro (robot description, xacro)
@@ -1,8 +1,12 @@
 <?xml version="1.0"?>
 <robot xmlns:xacro="http://www.ros.org/wiki/xacro" name="fd">
-    <!-- Import iiwa urdf file -->
-    <xacro:include filename="$(find fd_description)/urdf/fd.urdf" />
-    <!-- Import iiwa ros2_control description -->
+    <!-- Parameters -->
+    <xacro:arg name="robot_id" default="fd"/> <!-- Name of the haptic interface -->
+    <xacro:arg name="use_fake_hardware" default="false"/>
+    <!-- Import interface urdf file -->
+    <xacro:include filename="$(find fd_description)/urdf/fd.urdf.xacro"/>
+    <xacro:haptic_interface robot_id="$(arg robot_id)"/>
+    <!-- Import interface ros2_control description -->
     <xacro:include filename="$(find fd_description)/ros2_control/fd.r2c_hardware.xacro" />
-    <xacro:fd_ros2_control name="FDHapticInterface"/>
+    <xacro:fd_ros2_control plugin_name="FDHapticInterface" robot_id= "$(arg robot_id)" use_fake_hardware="$(arg use_fake_hardware)"/>
 </robot>

File: fd_description/ros2_control/fd.r2c_hardware.xacro (robot description, xacro)
@@ -1,28 +1,26 @@
 <?xml version="1.0"?>
 <robot xmlns:xacro="http://www.ros.org/wiki/xacro">
-    <xacro:macro name="fd_ros2_control" params="name">
-        <ros2_control name="${name}" type="system">
+    <xacro:macro name="fd_ros2_control" params="plugin_name robot_id use_fake_hardware">
+        <ros2_control name="${plugin_name}" type="system">
             <hardware>
-                <plugin>fd_hardware/FDEffortHardwareInterface</plugin>
-                <param name="interface_ID">-1</param>
+                <xacro:if value="${use_fake_hardware}">
+                    <plugin>fake_components/GenericSystem</plugin>
+                </xacro:if>
+                <xacro:unless value="${use_fake_hardware}">
+                    <plugin>fd_hardware/FDEffortHardwareInterface</plugin>
+                    <param name="interface_ID">-1</param>
+                </xacro:unless>
             </hardware>
-            <joint name="fd_x">
-                <command_interface name="effort" />
+            <xacro:macro name="configure_joint" params="joint_name">
+                <joint name="${joint_name}">
+                <command_interface name="effort"/>
                 <state_interface name="position"/>
                 <state_interface name="velocity"/>
                 <state_interface name="effort"/>
-            </joint>
-            <joint name="fd_y">
-                <command_interface name="effort" />
-                <state_interface name="position"/>
-                <state_interface name="velocity"/>
-                <state_interface name="effort"/>
-            </joint>
-            <joint name="fd_z">
-                <command_interface name="effort" />
-                <state_interface name="position"/>
-                <state_interface name="velocity"/>
-                <state_interface name="effort"/>
-            </joint>
+                </joint>
+            </xacro:macro>
+            <xacro:configure_joint joint_name="${robot_id}_x"/>
+            <xacro:configure_joint joint_name="${robot_id}_y"/>
+            <xacro:configure_joint joint_name="${robot_id}_z"/>
         </ros2_control>
     </xacro:macro>

Commit message: fd_description: orientation model + ros2 control HW config

File: fd_description/config/fd.config.xacro (robot description, xacro)
@@ -4,9 +4,10 @@
     <xacro:arg name="robot_id" default="fd"/> <!-- Name of the haptic interface -->
     <xacro:arg name="use_fake_hardware" default="false"/>
+    <xacro:arg name="use_orientation" default="false"/>
     <!-- Import interface urdf file -->
     <xacro:include filename="$(find fd_description)/urdf/fd.urdf.xacro"/>
-    <xacro:haptic_interface robot_id="$(arg robot_id)"/>
+    <xacro:haptic_interface robot_id="$(arg robot_id)" use_orientation="$(arg use_orientation)"/>
     <!-- Import interface ros2_control description -->
     <xacro:include filename="$(find fd_description)/ros2_control/fd.r2c_hardware.xacro" />
-    <xacro:fd_ros2_control plugin_name="FDHapticInterface" robot_id= "$(arg robot_id)" use_fake_hardware="$(arg use_fake_hardware)"/>
+    <xacro:fd_ros2_control robot_id= "$(arg robot_id)" use_fake_hardware="$(arg use_fake_hardware)" use_orientation="$(arg use_orientation)"/>
 </robot>

File: fd_description/ros2_control/fd.r2c_hardware.xacro (robot description, xacro)
@@ -1,5 +1,5 @@
 <?xml version="1.0"?>
 <robot xmlns:xacro="http://www.ros.org/wiki/xacro">
-    <xacro:macro name="fd_ros2_control" params="plugin_name robot_id use_fake_hardware">
+    <xacro:macro name="fd_ros2_control" params="robot_id plugin_name:='FDHapticInterface' use_fake_hardware:='false' use_orientation:=false">
         <ros2_control name="${plugin_name}" type="system">
             <hardware>
@@ -12,15 +12,28 @@
                 </xacro:unless>
             </hardware>
-            <xacro:macro name="configure_joint" params="joint_name">
+            <!-- Configure translations -->
+            <xacro:macro name="configure_translation_joint" params="joint_name">
                 <joint name="${joint_name}">
-                <command_interface name="effort"/>
-                <state_interface name="position"/>
-                <state_interface name="velocity"/>
-                <state_interface name="effort"/>
+                    <command_interface name="effort"/>
+                    <state_interface name="position"/>
+                    <state_interface name="velocity"/>
+                    <state_interface name="effort"/>
                 </joint>
             </xacro:macro>
-            <xacro:configure_joint joint_name="${robot_id}_x"/>
-            <xacro:configure_joint joint_name="${robot_id}_y"/>
-            <xacro:configure_joint joint_name="${robot_id}_z"/>
+            <xacro:configure_translation_joint joint_name="${robot_id}_x"/>
+            <xacro:configure_translation_joint joint_name="${robot_id}_y"/>
+            <xacro:configure_translation_joint joint_name="${robot_id}_z"/>
+            <!-- Configure orientation (read-only!) -->
+            <xacro:if value="${use_orientation}">
+                <xacro:macro name="configure_rotation_joint" params="joint_name">
+                    <joint name="${joint_name}">
+                        <state_interface name="position"/>
+                        <state_interface name="velocity"/>
+                    </joint>
+                </xacro:macro>
+                <xacro:configure_rotation_joint joint_name="${robot_id}_roll"/>
+                <xacro:configure_rotation_joint joint_name="${robot_id}_pitch"/>
+                <xacro:configure_rotation_joint joint_name="${robot_id}_yaw"/>
+            </xacro:if>
         </ros2_control>
     </xacro:macro>

File: fd_description/urdf/fd.urdf.xacro (robot description, xacro)
@@ -1,10 +1,14 @@
 <?xml version="1.0" encoding='utf-8'?>
 <robot xmlns:xacro="http://www.ros.org/wiki/xacro" name="fd">
-    <xacro:macro name="haptic_interface" params="robot_id:='fd'">
+    <xacro:macro name="haptic_interface" params="robot_id:='fd' use_orientation:='false'">
         <link name="${robot_id}_base"/>
         <link name="${robot_id}_x_link"/>
         <link name="${robot_id}_y_link"/>
         <link name="${robot_id}_z_link"/>
+        <link name="${robot_id}_roll_link"/>
+        <link name="${robot_id}_pitch_link"/>
+        <link name="${robot_id}_yaw_link"/>
         <link name="${robot_id}_ee"/>
+        <!-- Translation -->
         <joint name="${robot_id}_x" type="prismatic">
             <origin rpy="0 0 0" xyz="0 0 0"/>
@@ -28,7 +32,37 @@
             <limit effort="12" velocity="1.0" lower="-2" upper="2" />
         </joint>
-        <joint name="tool" type="fixed">
+        <!-- Orientation from XYZ roll-pitch-yaw angles -->
+        <!-- TODO: change when/if floating joints are supported by ros2 control AND KDL -->
+        <xacro:if value="${use_orientation}">
+            <xacro:property name="orientation_joint_type" value="revolute" />
+        </xacro:if>
+        <xacro:unless value="${use_orientation}">
+            <xacro:property name="orientation_joint_type" value="fixed" />
+        </xacro:unless>
+        <joint name="${robot_id}_roll" type="${orientation_joint_type}">
             <origin rpy="0 0 0" xyz="0 0 0"/>
             <parent link="${robot_id}_z_link"/>
+            <child link="${robot_id}_roll_link"/>
+            <axis xyz="1 0 0"/>
+            <limit effort="0.4" velocity="10.0" lower="-${pi}" upper="${pi}" />
+        </joint>
+        <joint name="${robot_id}_pitch" type="${orientation_joint_type}">
+            <origin rpy="0 0 0" xyz="0 0 0"/>
+            <parent link="${robot_id}_roll_link"/>
+            <child link="${robot_id}_pitch_link"/>
+            <axis xyz="0 1 0"/>
+            <limit effort="0.4" velocity="10.0" lower="-${pi}" upper="${pi}" />
+        </joint>
+        <joint name="${robot_id}_yaw" type="${orientation_joint_type}">
+            <origin rpy="0 0 0" xyz="0 0 0"/>
+            <parent link="${robot_id}_pitch_link"/>
+            <child link="${robot_id}_yaw_link"/>
+            <axis xyz="0 0 1"/>
+            <limit effort="0.4" velocity="10.0" lower="-${pi}" upper="${pi}" />
+        </joint>
+        <!-- Tool -->
+        <joint name="${robot_id}_tool" type="fixed">
+            <origin rpy="0 0 0" xyz="0 0 0"/>
+            <parent link="${robot_id}_yaw_link"/>
             <child link="${robot_id}_ee"/>
         </joint>

Commit message: feat: (fd_description) add optional clutch support

File: fd_description/config/fd.config.xacro (robot description, xacro)
@@ -5,9 +5,10 @@
     <xacro:arg name="use_fake_hardware" default="false"/>
     <xacro:arg name="use_orientation" default="false"/>
+    <xacro:arg name="use_clutch" default="false"/>
     <!-- Import interface urdf file -->
     <xacro:include filename="$(find fd_description)/urdf/fd.urdf.xacro"/>
-    <xacro:haptic_interface robot_id="$(arg robot_id)" use_orientation="$(arg use_orientation)"/>
+    <xacro:haptic_interface robot_id="$(arg robot_id)" use_orientation="$(arg use_orientation)" use_clutch="$(arg use_clutch)"/>
     <!-- Import interface ros2_control description -->
     <xacro:include filename="$(find fd_description)/ros2_control/fd.r2c_hardware.xacro" />
-    <xacro:fd_ros2_control robot_id= "$(arg robot_id)" use_fake_hardware="$(arg use_fake_hardware)" use_orientation="$(arg use_orientation)"/>
+    <xacro:fd_ros2_control robot_id= "$(arg robot_id)" use_fake_hardware="$(arg use_fake_hardware)" use_orientation="$(arg use_orientation)" use_clutch="$(arg use_clutch)"/>
 </robot>

File: fd_description/ros2_control/fd.r2c_hardware.xacro (robot description, xacro)
@@ -1,5 +1,5 @@
 <?xml version="1.0"?>
 <robot xmlns:xacro="http://www.ros.org/wiki/xacro">
-    <xacro:macro name="fd_ros2_control" params="robot_id plugin_name:='FDHapticInterface' use_fake_hardware:='false' use_orientation:=false">
+    <xacro:macro name="fd_ros2_control" params="robot_id plugin_name:='FDHapticInterface' use_fake_hardware:='false' use_orientation:=false use_clutch:='false'">
         <ros2_control name="${plugin_name}" type="system">
             <hardware>
@@ -36,4 +36,8 @@
                 <xacro:configure_rotation_joint joint_name="${robot_id}_yaw"/>
             </xacro:if>
+            <!-- Configure clutch -->
+            <xacro:if value="${use_clutch}">
+                <xacro:configure_translation_joint joint_name="${robot_id}_clutch"/>
+            </xacro:if>
         </ros2_control>
     </xacro:macro>

File: fd_description/urdf/fd.urdf.xacro (robot description, xacro)
@@ -1,5 +1,5 @@
 <?xml version="1.0" encoding='utf-8'?>
 <robot xmlns:xacro="http://www.ros.org/wiki/xacro" name="fd">
-    <xacro:macro name="haptic_interface" params="robot_id:='fd' use_orientation:='false'">
+    <xacro:macro name="haptic_interface" params="robot_id:='fd' use_orientation:='false' use_clutch:='false'">
         <link name="${robot_id}_base"/>
         <link name="${robot_id}_x_link"/>
@@ -67,4 +67,15 @@
             <child link="${robot_id}_ee"/>
         </joint>
+        <!-- Clutch -->
+        <xacro:if value="${use_clutch}">
+            <link name="${robot_id}_virtual_clutch_link"/>
+            <joint name="${robot_id}_clutch" type="prismatic">
+                <origin rpy="0 0 0" xyz="0 0 0"/>
+                <parent link="${robot_id}_ee"/>
+                <child link="${robot_id}_clutch"/>
+                <axis xyz="1 0 0"/>
+            <limit effort="12" velocity="1.0" lower="-0.05" upper="0.05" />
+        </joint>
+        </xacro:if>
     </xacro:macro>
 </robot>

Commit message: fix: fd_HW compatibility + errors fixes
- Typo "fd_clucth" link
- Add "orientation_is_actuated" parameters in r2c xacro
- In "config" xacro, make "orientation_is_actuated" = "use_orientation"
for compatibility reasons (fd_HW tests do not allow the alternative)

- TODO: Make "use_clutch" invalid when thge rotation is not defined ->
take interface name as global param to define allowed combinations ?!

File: fd_description/config/fd.config.xacro (robot description, xacro)
@@ -8,7 +8,17 @@
     <!-- Import interface urdf file -->
     <xacro:include filename="$(find fd_description)/urdf/fd.urdf.xacro"/>
-    <xacro:haptic_interface robot_id="$(arg robot_id)" use_orientation="$(arg use_orientation)" use_clutch="$(arg use_clutch)"/>
-    <!-- Import interface ros2_control description -->
+    <xacro:haptic_interface
+    	robot_id="$(arg robot_id)"
+    	use_orientation="$(arg use_orientation)"
+    	use_clutch="$(arg use_clutch)"
+    />
+    <!-- Import and setup interface ros2_control description -->
     <xacro:include filename="$(find fd_description)/ros2_control/fd.r2c_hardware.xacro" />
-    <xacro:fd_ros2_control robot_id= "$(arg robot_id)" use_fake_hardware="$(arg use_fake_hardware)" use_orientation="$(arg use_orientation)" use_clutch="$(arg use_clutch)"/>
+    <xacro:fd_ros2_control
+        robot_id= "$(arg robot_id)"
+        use_fake_hardware="$(arg use_fake_hardware)"
+        use_orientation="$(arg use_orientation)"
+    	orientation_is_actuated="$(arg use_orientation)"
+        use_clutch="$(arg use_clutch)"
+    /> <!-- orientation_is_actuated = use_orientation for now (see HW impl.) -->
 </robot>

File: fd_description/ros2_control/fd.r2c_hardware.xacro (robot description, xacro)
@@ -1,5 +1,5 @@
 <?xml version="1.0"?>
 <robot xmlns:xacro="http://www.ros.org/wiki/xacro">
-    <xacro:macro name="fd_ros2_control" params="robot_id plugin_name:='FDHapticInterface' use_fake_hardware:='false' use_orientation:=false use_clutch:='false'">
+    <xacro:macro name="fd_ros2_control" params="robot_id plugin_name:='FDHapticInterface' use_fake_hardware:='false' use_orientation:='false' orientation_is_actuated:='false' use_clutch:='false'">
         <ros2_control name="${plugin_name}" type="system">
             <hardware>
@@ -30,4 +30,8 @@
                         <state_interface name="position"/>
                         <state_interface name="velocity"/>
+                        <xacro:if value="${orientation_is_actuated}">
+                            <state_interface name="effort"/>
+                            <command_interface name="effort"/>
+                        </xacro:if>
                     </joint>
                 </xacro:macro>

File: fd_description/urdf/fd.urdf.xacro (robot description, xacro)
@@ -73,5 +73,5 @@
                 <origin rpy="0 0 0" xyz="0 0 0"/>
                 <parent link="${robot_id}_ee"/>
-                <child link="${robot_id}_clutch"/>
+                <child link="${robot_id}_virtual_clutch_link"/>
                 <axis xyz="1 0 0"/>
             <limit effort="12" velocity="1.0" lower="-0.05" upper="0.05" />

Commit message: More flexible fd interface modelling and control (#6)
* add: fake hardware tags and robot_id parameters in urdf

Add:
 - 'use_fake_hardware' xacro arg
 - 'robot_id' xacro arg
 - 'plugin_name' xacro arg

* fd_description: orientation model + ros2 control HW config

* feat: (fd_description) add optional clutch support

* fix: fd_HW compatibility + errors fixes

- Typo "fd_clucth" link
- Add "orientation_is_actuated" parameters in r2c xacro
- In "config" xacro, make "orientation_is_actuated" = "use_orientation"
for compatibility reasons (fd_HW tests do not allow the alternative)

- TODO: Make "use_clutch" invalid when thge rotation is not defined ->
take interface name as global param to define allowed combinations ?!

* launch fix: use clutch by default

* feat repare demo :
 - remove ee_broadcaster from demo
 - fix config fd controller

---------

Co-authored-by: Thibault Poignonec <thibault.poignonec@lirmm.fr>

File: fd_description/config/fd.config.xacro (robot description, xacro)
@@ -1,8 +1,24 @@
 <?xml version="1.0"?>
 <robot xmlns:xacro="http://www.ros.org/wiki/xacro" name="fd">
-    <!-- Import iiwa urdf file -->
-    <xacro:include filename="$(find fd_description)/urdf/fd.urdf" />
-    <!-- Import iiwa ros2_control description -->
+    <!-- Parameters -->
+    <xacro:arg name="robot_id" default="fd"/> <!-- Name of the haptic interface -->
+    <xacro:arg name="use_fake_hardware" default="false"/>
+    <xacro:arg name="use_orientation" default="false"/>
+    <xacro:arg name="use_clutch" default="false"/>
+    <!-- Import interface urdf file -->
+    <xacro:include filename="$(find fd_description)/urdf/fd.urdf.xacro"/>
+    <xacro:haptic_interface
+    	robot_id="$(arg robot_id)"
+    	use_orientation="$(arg use_orientation)"
+    	use_clutch="$(arg use_clutch)"
+    />
+    <!-- Import and setup interface ros2_control description -->
     <xacro:include filename="$(find fd_description)/ros2_control/fd.r2c_hardware.xacro" />
-    <xacro:fd_ros2_control name="FDHapticInterface"/>
+    <xacro:fd_ros2_control
+        robot_id= "$(arg robot_id)"
+        use_fake_hardware="$(arg use_fake_hardware)"
+        use_orientation="$(arg use_orientation)"
+    	orientation_is_actuated="$(arg use_orientation)"
+        use_clutch="$(arg use_clutch)"
+    /> <!-- orientation_is_actuated = use_orientation for now (see HW impl.) -->
 </robot>

File: fd_description/ros2_control/fd.r2c_hardware.xacro (robot description, xacro)
@@ -1,28 +1,47 @@
 <?xml version="1.0"?>
 <robot xmlns:xacro="http://www.ros.org/wiki/xacro">
-    <xacro:macro name="fd_ros2_control" params="name">
-        <ros2_control name="${name}" type="system">
+    <xacro:macro name="fd_ros2_control" params="robot_id plugin_name:='FDHapticInterface' use_fake_hardware:='false' use_orientation:='false' orientation_is_actuated:='false' use_clutch:='false'">
+        <ros2_control name="${plugin_name}" type="system">
             <hardware>
-                <plugin>fd_hardware/FDEffortHardwareInterface</plugin>
-                <param name="interface_ID">-1</param>
+                <xacro:if value="${use_fake_hardware}">
+                    <plugin>fake_components/GenericSystem</plugin>
+                </xacro:if>
+                <xacro:unless value="${use_fake_hardware}">
+                    <plugin>fd_hardware/FDEffortHardwareInterface</plugin>
+                    <param name="interface_ID">-1</param>
+                </xacro:unless>
             </hardware>
-            <joint name="fd_x">
-                <command_interface name="effort" />
-                <state_interface name="position"/>
-                <state_interface name="velocity"/>
-                <state_interface name="effort"/>
-            </joint>
-            <joint name="fd_y">
-                <command_interface name="effort" />
-                <state_interface name="position"/>
-                <state_interface name="velocity"/>
-                <state_interface name="effort"/>
-            </joint>
-            <joint name="fd_z">
-                <command_interface name="effort" />
-                <state_interface name="position"/>
-                <state_interface name="velocity"/>
-                <state_interface name="effort"/>
-            </joint>
+            <!-- Configure translations -->
+            <xacro:macro name="configure_translation_joint" params="joint_name">
+                <joint name="${joint_name}">
+                    <command_interface name="effort"/>
+                    <state_interface name="position"/>
+                    <state_interface name="velocity"/>
+                    <state_interface name="effort"/>
+                </joint>
+            </xacro:macro>
+            <xacro:configure_translation_joint joint_name="${robot_id}_x"/>
+            <xacro:configure_translation_joint joint_name="${robot_id}_y"/>
+            <xacro:configure_translation_joint joint_name="${robot_id}_z"/>
+            <!-- Configure orientation (read-only!) -->
+            <xacro:if value="${use_orientation}">
+                <xacro:macro name="configure_rotation_joint" params="joint_name">
+                    <joint name="${joint_name}">
+                        <state_interface name="position"/>
+                        <state_interface name="velocity"/>
+                        <xacro:if value="${orientation_is_actuated}">
+                            <state_interface name="effort"/>
+                            <command_interface name="effort"/>
+                        </xacro:if>
+                    </joint>
+                </xacro:macro>
+                <xacro:configure_rotation_joint joint_name="${robot_id}_roll"/>
+                <xacro:configure_rotation_joint joint_name="${robot_id}_pitch"/>
+                <xacro:configure_rotation_joint joint_name="${robot_id}_yaw"/>
+            </xacro:if>
+            <!-- Configure clutch -->
+            <xacro:if value="${use_clutch}">
+                <xacro:configure_translation_joint joint_name="${robot_id}_clutch"/>
+            </xacro:if>
         </ros2_control>
     </xacro:macro>
