Commit message: add button

File: fd_description/ros2_control/fd.r2c_hardware.xacro (robot description, xacro)
@@ -25,4 +25,10 @@
                 <state_interface name="effort"/>
             </joint>
+            <joint name="button">
+                <command_interface name="effort" />
+                <state_interface name="position"/>
+                <state_interface name="velocity"/>
+                <state_interface name="effort"/>
+            </joint>
         </ros2_control>
     </xacro:macro>

File: fd_description/urdf/fd.urdf (robot description, URDF)
Before this commit: robot fd, 5 links, 4 joints
Links:
- added link button_link
Joints:
- added joint button: type prismatic, parent fd_base, child button_link, origin xyz=0 0 0 rpy=0 0 0, axis 0 1 0, limit lower=-2 upper=2 effort=1 velocity=1.0

Commit message: change button type as gpio

File: fd_description/ros2_control/fd.r2c_hardware.xacro (robot description, xacro)
@@ -25,10 +25,7 @@
                 <state_interface name="effort"/>
             </joint>
-            <joint name="button">
-                <command_interface name="effort" />
+            <gpio name="button">
                 <state_interface name="position"/>
-                <state_interface name="velocity"/>
-                <state_interface name="effort"/>
-            </joint>
+    	    </gpio>
         </ros2_control>
     </xacro:macro>

File: fd_description/urdf/fd.urdf (robot description, URDF)
Before this commit: robot fd, 6 links, 5 joints
Links:
- removed link button_link
Joints:
- removed joint button

Commit message: update description file

File: fd_description/ros2_control/fd.r2c_hardware.xacro (robot description, xacro)
@@ -1,5 +1,7 @@
 <?xml version="1.0"?>
 <robot xmlns:xacro="http://www.ros.org/wiki/xacro">
-    <xacro:macro name="fd_ros2_control" params="robot_id plugin_name:='FDHapticInterface' use_fake_hardware:='false' use_orientation:='false' orientation_is_actuated:='false' use_clutch:='false'">
+    <xacro:macro
+        name="fd_ros2_control"
+        params="robot_id plugin_name:='FDHapticInterface' interface_id:='-1' use_fake_hardware:='false' use_orientation:='false' orientation_is_actuated:='false' use_clutch:='false' emulate_button:='true'">
         <ros2_control name="${plugin_name}" type="system">
             <hardware>
@@ -9,5 +11,7 @@
                 <xacro:unless value="${use_fake_hardware}">
                     <plugin>fd_hardware/FDEffortHardwareInterface</plugin>
-                    <param name="interface_ID">-1</param>
+                    <param name="interface_id">${interface_id}</param>
+                    <param name="emulate_button">${emulate_button}</param>
+                    <param name="inertia_interface_name">fd_inertia</param>
                 </xacro:unless>
             </hardware>

Commit message: Emulate button, cleanup parameters and logging (#25)
* add debug logs

* add parameters for emulate_button and interface_id

* make fd_inertia a parameter also

* emulate button

* update description file

* linting

* cleanup logging

File: fd_description/ros2_control/fd.r2c_hardware.xacro (robot description, xacro)
@@ -1,5 +1,7 @@
 <?xml version="1.0"?>
 <robot xmlns:xacro="http://www.ros.org/wiki/xacro">
-    <xacro:macro name="fd_ros2_control" params="robot_id plugin_name:='FDHapticInterface' use_fake_hardware:='false' use_orientation:='false' orientation_is_actuated:='false' use_clutch:='false'">
+    <xacro:macro
+        name="fd_ros2_control"
+        params="robot_id plugin_name:='FDHapticInterface' interface_id:='-1' use_fake_hardware:='false' use_orientation:='false' orientation_is_actuated:='false' use_clutch:='false' emulate_button:='false'">
         <ros2_control name="${plugin_name}" type="system">
             <hardware>
@@ -9,5 +11,7 @@
                 <xacro:unless value="${use_fake_hardware}">
                     <plugin>fd_hardware/FDEffortHardwareInterface</plugin>
-                    <param name="interface_ID">-1</param>
+                    <param name="interface_id">${interface_id}</param>
+                    <param name="emulate_button">${emulate_button}</param>
+                    <param name="inertia_interface_name">fd_inertia</param>
                 </xacro:unless>
             </hardware>
